Commit message: Replaced STL files by DAE and meshes cleaning

File: pf_description/urdf/r2000.urdf.xacro (robot description, xacro)
@@ -4,13 +4,13 @@
         <link name="${prefix}base_link" >
             <visual>
-                <origin xyz="0 0 0" rpy="1.57 0 1.57" />
+                <origin xyz="0 0 0" rpy="0 0 0" />
                 <geometry>
-                    <mesh filename="package://pf_description/meshes/R2000.stl" scale="0.001 0.001 0.001" />
+                    <mesh filename="$(find pf_description)/meshes/R2000.dae" />
                 </geometry>
             </visual>
             <collision>
-                <origin xyz="0 0 0.045" rpy="0 0 0" />
+                <origin xyz="-0.0058 0 -0.03885" rpy="0 0 0" />
                 <geometry>
-                    <box size="0.108 0.118 0.128" />
+                    <box size="0.118 0.108 0.117" />
                 </geometry>
             </collision>

File: pf_description/urdf/r2300.urdf.xacro (robot description, xacro)
@@ -4,13 +4,13 @@
         <link name="${prefix}base_link" >
             <visual>
-                <origin xyz="-0.00195 0.0158 -0.0094" rpy="-1.57 0 1.57" />
+                <origin xyz="0 0 0" rpy="0 0 0" />
                 <geometry>
-                    <mesh filename="package://pf_description/meshes/R2300.stl" scale="0.001 0.001 0.001" />
+                    <mesh filename="$(find pf_description)/meshes/R2300.dae" />
                 </geometry>
             </visual>
             <collision>
-                <origin xyz="-0.00195 0.0158 -0.0094" rpy="-1.57 0 1.57" />
+                <origin xyz="0.01195 0.0158 -0.017" rpy="0 0 0" />
                 <geometry>
-                    <box size="0.0951 0.0685 0.0695" />
+                    <box size="0.07 0.0959 0.0586" />
                 </geometry>
             </collision>
